Commit message: gait clock rew

File: assets/officialdesign/OFFICIALdesign/urdf/OFFICIALdesign.urdf (robot description, URDF)
Before this commit: robot OFFICIALdesign, 13 links, 12 joints
Joints:
- joint Bubleft_joint: limit lower=-0.20943951023931956 upper=0.20943951023931956 effort=10.3 velocity=4.7 -> lower=-0.20943951023931956 upper=0.20943951023931956 effort=11.77 velocity=2.31
- joint Bubright_joint: limit lower=-0.20943951023931956 upper=0.20943951023931956 effort=10.3 velocity=4.7 -> lower=-0.20943951023931956 upper=0.20943951023931956 effort=11.77 velocity=2.31
- joint Hipleft_joint: limit lower=-0.2617993877991494 upper=0.7853981633974483 effort=10.3 velocity=4.7 -> lower=-0.2617993877991494 upper=0.7853981633974483 effort=11.77 velocity=2.31
- joint Hipright_joint: limit lower=-0.7853981633974483 upper=0.2617993877991494 effort=10.3 velocity=4.7 -> lower=-0.7853981633974483 upper=0.2617993877991494 effort=11.77 velocity=2.31
- joint Kneeleft_joint: limit lower=-1.3089969389957472 upper=0.0 effort=10.3 velocity=4.7 -> lower=-1.3089969389957472 upper=0.0 effort=11.77 velocity=2.31
- joint Kneeright: limit lower=0.0 upper=1.3089969389957472 effort=10.3 velocity=4.7 -> lower=0.0 upper=1.3089969389957472 effort=11.77 velocity=2.31
